Commit message: further improvisations for cameralink

File: Assignment_2/src/custom_arm_description/urdf/custom_arm.urdf.xacro (robot description, xacro)
@@ -16,5 +16,5 @@
   <xacro:arg name="external_urdf_loc"               default=""/>
   <xacro:arg name="hardware_type"                   default="actual"/>
-  <xacro:property name="mesh_directory"             value="package://interbotix_xsarm_descriptions/meshes/${robot_model}_meshes"/>
+  <xacro:property name="mesh_directory"             value="package://custom_arm_description/meshes/${robot_model}_meshes"/>
   <xacro:property name="urdf_loc"                   value="$(arg external_urdf_loc)"/>
   <xacro:property name="hardware_type"              value="$(arg hardware_type)"/>
@@ -46,5 +46,5 @@
   <xacro:property name="finger_limit_vel"           value="1"/>
   <material name="interbotix_black">
-    <texture filename="package://interbotix_xsarm_descriptions/meshes/interbotix_black.png"/>
+    <texture filename="package://custom_arm_description/meshes/interbotix_black.png"/>
   </material>
   <xacro:if value="$(arg use_world_frame)">
@@ -312,5 +312,5 @@
   <link name="camera_color_optical_frame"/>
   <joint name="wrist_to_camera_optical" type="fixed">
-    <origin xyz="0.05 0 0.10" rpy="0 0 0"/>
+    <origin xyz="0.0 0 0.0" rpy="0 0 0.785"/>
     <parent link="$(arg robot_name)/wrist_link"/>
     <child link="camera_color_optical_frame"/>
@@ -448,5 +448,5 @@
     <!-- If the AR tag is being used, then add the AR tag mount -->
     <xacro:if value="$(arg show_ar_tag)">
-      <xacro:include filename="$(find interbotix_xsarm_descriptions)/urdf/ar_tag.urdf.xacro"/>
+      <xacro:include filename="$(find custom_arm_description)/urdf/ar_tag.urdf.xacro"/>
     </xacro:if> <!-- show_ar_tag -->
     <!-- If the gripper bar is being used, then also add the gripper bar -->
@@ -661,6 +661,6 @@
     </xacro:if> <!-- show_gripper_bar -->
   </xacro:if> <!-- use_gripper -->
-  <xacro:include filename="$(find interbotix_xsarm_descriptions)/urdf/control.urdf.xacro"/>
-  <xacro:include filename="$(find interbotix_xsarm_descriptions)/urdf/gazebo_configs.urdf.xacro"/>
+  <xacro:include filename="$(find custom_arm_description)/urdf/control.urdf.xacro"/>
+  <xacro:include filename="$(find custom_arm_description)/urdf/gazebo_configs.urdf.xacro"/>
   <xacro:if value="${hardware_type == 'gz_classic'}">
     <xacro:gazebo_configs/>
